Commit message: fix frame issues

File: catkin_ws/src/slam_project/urdf/udacity_bot.xacro (robot description, xacro)
@@ -135,5 +135,5 @@
   </link>
   <!-- Camera Link -->
-  <link name="camera">
+  <link name="camera_link">
     <inertial>
       <mass value="0.1"/>
@@ -161,4 +161,10 @@
     </collision>
   </link>
+  <link name="camera_rgbd_frame" type="fixed"></link>
+  <joint name="camera_rgbd_joint" type="fixed">
+    <origin xyz="0 0 0" rpy="-1.5707 0 -1.5707" />
+    <parent link="camera_link" />
+    <child link="camera_rgbd_frame"/>
+  </joint>
   <!-- Hokuyo Link -->
   <link name="hokuyo">
@@ -204,5 +210,5 @@
   <joint type="fixed" name="camera_joint">
     <origin xyz="0.2 0 0" rpy="0 0 0"/>
-    <child link="camera"/>
+    <child link="camera_link"/>
     <parent link="chassis"/>
   </joint>

Commit message: progress

File: catkin_ws/src/slam_project/urdf/udacity_bot.xacro (robot description, xacro)
@@ -135,5 +135,5 @@
   </link>
   <!-- Camera Link -->
-  <link name="camera_link">
+  <link name="camera">
     <inertial>
       <mass value="0.1"/>
@@ -164,5 +164,5 @@
   <joint name="camera_rgbd_joint" type="fixed">
     <origin xyz="0 0 0" rpy="-1.5707 0 -1.5707" />
-    <parent link="camera_link" />
+    <parent link="camera" />
     <child link="camera_rgbd_frame"/>
   </joint>
@@ -210,5 +210,5 @@
   <joint type="fixed" name="camera_joint">
     <origin xyz="0.2 0 0" rpy="0 0 0"/>
-    <child link="camera_link"/>
+    <child link="camera"/>
     <parent link="chassis"/>
   </joint>

Commit message: refactor

File: catkin_ws/src/slam_project/urdf/udacity_bot.xacro (robot description, xacro)
@@ -1,5 +1,5 @@
 <?xml version='1.0'?>
-<robot name="my_bot" xmlns:xacro="http://www.ros.org/wiki/xacro">
-<xacro:include filename="$(find slam_project)/urdf/my_bot.gazebo" />
+<robot name="udacity_bot" xmlns:xacro="http://www.ros.org/wiki/xacro">
+<xacro:include filename="$(find slam_project)/urdf/udacity_bot.gazebo" />
   <link name="robot_footprint"></link>
   <joint name="robot_footprint_joint" type="fixed">
@@ -98,5 +98,5 @@
       </geometry>
     </collision>
- </link>
+  </link>
   <link name="left_wheel">
     <visual>
@@ -115,12 +115,12 @@
       />
     </inertial>
-	<collision>
-      <origin xyz="0 0 0" rpy="0 1.5707 1.5707"/>
-       <geometry>
-        <cylinder length="0.025" radius="0.06"/>
-      </geometry>
-    </collision>
-  </link>
-<joint type="continuous" name="left_wheel_hinge">
+    <collision>
+      <origin xyz="0 0 0" rpy="0 1.5707 1.5707"/>
+       <geometry>
+        <cylinder length="0.025" radius="0.06"/>
+      </geometry>
+    </collision>
+  </link>
+  <joint type="continuous" name="left_wheel_hinge">
     <origin xyz="0 0.226 0" rpy="0 0 0"/>
     <child link="left_wheel"/>
@@ -130,5 +130,5 @@
     <joint_properties damping="1.0" friction="1.0"/>
   </joint>
-<joint type="continuous" name="right_wheel_hinge">
+  <joint type="continuous" name="right_wheel_hinge">
     <origin xyz="0 -0.226 0" rpy="0 0 0"/>
     <child link="right_wheel"/>
@@ -138,5 +138,5 @@
     <joint_properties damping="1.0" friction="1.0"/>
   </joint>
-<link name="camera_link">
+  <link name="camera_link">
      <visual>
       <origin xyz="0 0 0" rpy="0 0 0"/>
@@ -160,5 +160,5 @@
       </geometry>
     </collision>
-</link>
+  </link>
   <joint name="camera_joint" type="fixed">
     <origin xyz="0.1 0 0.1" rpy="0 0 0" />
@@ -166,5 +166,5 @@
     <child link="camera_link"/>
   </joint>
-<link name="camera_rgbd_frame">
+  <link name="camera_rgbd_frame">
      <visual>
       <origin xyz="0 0 0" rpy="0 0 0"/>
@@ -188,11 +188,11 @@
       </geometry>
     </collision>
-</link>
+  </link>
   <joint name="rgbd_joint" type="fixed">
-    <origin xyz="0.1 0 0.1" rpy="-1.5707 0  -1.5707" />
-    <parent link="chassis"/>
+    <origin xyz="0 0 -0.05" rpy="-1.5707 0  -1.5707" />
+    <parent link="camera_link"/>
     <child link="camera_rgbd_frame"/>
   </joint>
-<link name="hokuyo">
+  <link name="hokuyo">
      <visual>
       <origin xyz="0 0 0" rpy="0 0 0"/>
@@ -216,9 +216,9 @@
       </geometry>
     </collision>
-</link>
+  </link>
   <joint name="hokuyo_joint" type="fixed">
     <origin xyz=".1 0 .16 " rpy="0 0 0" />
     <parent link="chassis"/>
     <child link="hokuyo"/>
-</joint>
+  </joint>
 </robot>
